File: PCB/alim_hat/alim_hat.sch (KiCad schematic (older format))
At the start: 42 parts, among them J1 Screw_Terminal_01x04, J10 Conn_01x02, J11 Conn_01x02, J12 Conn_01x02, J2 Barrel_Jack_MountingPin, J3 Conn_02x04_Odd_Even, J4 Jack-DC, J5 Jack-DC, J6 Jack-DC, J7 Jack-DC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

Commit message: add  lcls part number and add Fab file
Parts:
- removed J2: Barrel_Jack_MountingPin, Connector_BarrelJack:BarrelJack_Horizontal, symbol Connector:Barrel_Jack_MountingPin
- added J2: Jack-DC, Connector_BarrelJack:BarrelJack_Horizontal, symbol Connector:Jack-DC
- C1, C2: LCSC (none) -> C311622
- D1: LCSC (none) -> C134429
- F1: LCSC (none) -> C151162
- F2, F3, F4, F5: LCSC (none) -> C207091
- R1, R2, R3, R4: value 0.02 -> 0.02 1W; footprint Resistor_SMD:R_2010_5025Metric -> Resistor_SMD:R_2512_6332Metric; LCSC (none) -> C127705
- R10, R11, R12, R5, R6, R7, R8, R9: LCSC (none) -> C17414
- U1, U2, U3, U4: LCSC (none) -> C138706
Changed lines of the file:
@@
-$EndComp
-$Comp
-L Connector:Barrel_Jack_MountingPin J2
-U 1 1 5E5C7127
-P 9850 2250
-F 0 "J2" H 9907 2567 50  0000 C CNN
-F 1 "Barrel_Jack_MountingPin" H 9550 2500 50  0000 C CNN
-F 2 "Connector_BarrelJack:BarrelJack_Horizontal" H 9900 2210 50  0001 C CNN
-F 3 "~" H 9900 2210 50  0001 C CNN
-	1    9850 2250
-	-1   0    0    -1
 $EndComp
 $Comp
@@
 $EndComp
 $Comp
-L power:GND #PWR0102
-U 1 1 5E5C7139
-P 9850 2550
-F 0 "#PWR0102" H 9850 2300 50  0001 C CNN
-F 1 "GND" H 9855 2377 50  0000 C CNN
-F 2 "" H 9850 2550 50  0001 C CNN
-F 3 "" H 9850 2550 50  0001 C CNN
-	1    9850 2550
-	-1   0    0    -1
-$EndComp
-$Comp
 L power:GND #PWR0103
 U 1 1 5E5C713F
@@
 F 2 "Diode_SMD:D_SOD-123" H 9150 2200 50  0001 C CNN
 F 3 "~" H 9150 2200 50  0001 C CNN
+F 4 "C134429" V 9150 2200 50  0001 C CNN "LCSC"
 	1    9150 2200
 	0    1    1    0
@@
 F 2 "fuse:FUSC3216X100N" H 9200 1750 50  0001 L CNN
 F 3 "~" H 9150 1950 50  0001 C CNN
+F 4 "C151162" H 9150 1950 50  0001 C CNN "LCSC"
 	1    9150 1950
 	1    0    0    -1
@@
 F 2 "capa:CAPAE660X800N" H 8138 5400 50  0001 C CNN
 F 3 "~" H 8100 5550 50  0001 C CNN
+F 4 "C311622" H 8100 5550 50  0001 C CNN "LCSC"
 	1    8100 5550
 	1    0    0    -1
@@
 F 2 "capa:CAPAE660X800N" H 10588 5400 50  0001 C CNN
 F 3 "~" H 10550 5550 50  0001 C CNN
+F 4 "C311622" H 10550 5550 50  0001 C CNN "LCSC"
 	1    10550 5550
 	1    0    0    -1
@@
 $EndComp
 Wire Wire Line
-	8650 5550 8850 5550
-Wire Wire Line
 	8100 5400 8500 5400
 Wire Wire Line
@@
 	8100 5700 8650 5700
 Connection ~ 8100 5700
-Wire Wire Line
-	8650 5550 8650 5700
 Wire Wire Line
 	9950 5450 10300 5450
@@
 F 2 "fuse:THRMC7451X160N" H 3000 5500 50  0001 L CNN
 F 3 "~" H 2950 5700 50  0001 C CNN
+F 4 "C207091" V 2950 5700 50  0001 C CNN "LCSC"
 	1    2950 5700
 	0    1    1    0
@@
 F 2 "Package_SO:SOIC-8_3.9x4.9mm_P1.27mm" H 3100 5750 50  0001 C CNN
 F 3 "http://www.ti.com/lit/ds/symlink/ina219.pdf" H 2650 6000 50  0001 C CNN
+F 4 "C138706" V 2300 6100 50  0001 C CNN "LCSC"
 	1    2300 6100
 	0    1    1    0
@@
 AR Path="/5E5E1120" Ref="R3"  Part="1"
 F 0 "R3" V 2093 5600 50  0000 C CNN
-F 1 "0.02" V 2184 5600 50  0000 C CNN
-F 2 "Resistor_SMD:R_2010_5025Metric" V 2230 5600 50  0001 C CNN
+F 1 "0.02 1W" V 2184 5600 50  0000 C CNN
+F 2 "Resistor_SMD:R_2512_6332Metric" V 2230 5600 50  0001 C CNN
 F 3 "~" H 2300 5600 50  0001 C CNN
+F 4 "C127705" V 2300 5600 50  0001 C CNN "LCSC"
 	1    2300 5600
 	0    1    1    0
@@
 F 2 "Resistor_SMD:R_0805_2012Metric" V 2430 6750 50  0001 C CNN
 F 3 "~" H 2500 6750 50  0001 C CNN
+F 4 "C17414" H 2500 6750 50  0001 C CNN "LCSC"
 	1    2500 6750
 	1    0    0    -1
@@
 F 2 "Resistor_SMD:R_0805_2012Metric" V 2330 6750 50  0001 C CNN
 F 3 "~" H 2400 6750 50  0001 C CNN
+F 4 "C17414" H 2400 6750 50  0001 C CNN "LCSC"
 	1    2400 6750
 	-1   0    0    1
@@
 F 2 "fuse:THRMC7451X160N" H 2950 3650 50  0001 L CNN
 F 3 "~" H 2900 3850 50  0001 C CNN
+F 4 "C207091" V 2900 3850 50  0001 C CNN "LCSC"
 	1    2900 3850
-	0    1    1    0
-$EndComp
-$Comp
-L Analog_ADC:INA219AxD U?
-U 1 1 5E5E1165
-P 2250 4250
-AR Path="/5E5C0CC9/5E5E1165" Ref="U?"  Part="1"
-AR Path="/5E5E1165" Ref="U1"  Part="1"
-F 0 "U1" V 2400 4650 50  0000 C CNN
-F 1 "INA219AxD" V 2500 4750 50  0000 C CNN
-F 2 "Package_SO:SOIC-8_3.9x4.9mm_P1.27mm" H 3050 3900 50  0001 C CNN
-F 3 "http://www.ti.com/lit/ds/symlink/ina219.pdf" H 2600 4150 50  0001 C CNN
-	1    2250 4250
 	0    1    1    0
 $EndComp
@@
 AR Path="/5E5E117A" Ref="R1"  Part="1"
 F 0 "R1" V 2043 3750 50  0000 C CNN
-F 1 "0.02" V 2134 3750 50  0000 C CNN
-F 2 "Resistor_SMD:R_2010_5025Metric" V 2180 3750 50  0001 C CNN
+F 1 "0.02 1W" V 2134 3750 50  0000 C CNN
+F 2 "Resistor_SMD:R_2512_6332Metric" V 2180 3750 50  0001 C CNN
 F 3 "~" H 2250 3750 50  0001 C CNN
+F 4 "C127705" V 2250 3750 50  0001 C CNN "LCSC"
 	1    2250 3750
 	0    1    1    0
@@
 F 2 "Resistor_SMD:R_0805_2012Metric" V 2380 4900 50  0001 C CNN
 F 3 "~" H 2450 4900 50  0001 C CNN
+F 4 "C17414" H 2450 4900 50  0001 C CNN "LCSC"
 	1    2450 4900
 	1    0    0    -1
@@
 F 2 "Resistor_SMD:R_0805_2012Metric" V 2280 4900 50  0001 C CNN
 F 3 "~" H 2350 4900 50  0001 C CNN
+F 4 "C17414" H 2350 4900 50  0001 C CNN "LCSC"
 	1    2350 4900
 	-1   0    0    1
@@
 F 2 "fuse:THRMC7451X160N" H 5750 5500 50  0001 L CNN
 F 3 "~" H 5700 5700 50  0001 C CNN
+F 4 "C207091" V 5700 5700 50  0001 C CNN "LCSC"
 	1    5700 5700
 	0    1    1    0
@@
 F 2 "Package_SO:SOIC-8_3.9x4.9mm_P1.27mm" H 5850 5750 50  0001 C CNN
 F 3 "http://www.ti.com/lit/ds/symlink/ina219.pdf" H 5400 6000 50  0001 C CNN
+F 4 "C138706" V 5050 6100 50  0001 C CNN "LCSC"
 	1    5050 6100
 	0    1    1    0
@@
 AR Path="/5E5E11DA" Ref="R4"  Part="1"
 F 0 "R4" V 4843 5600 50  0000 C CNN
-F 1 "0.02" V 4934 5600 50  0000 C CNN
-F 2 "Resistor_SMD:R_2010_5025Metric" V 4980 5600 50  0001 C CNN
+F 1 "0.02 1W" V 4934 5600 50  0000 C CNN
+F 2 "Resistor_SMD:R_2512_6332Metric" V 4980 5600 50  0001 C CNN
 F 3 "~" H 5050 5600 50  0001 C CNN
+F 4 "C127705" V 5050 5600 50  0001 C CNN "LCSC"
 	1    5050 5600
 	0    1    1    0
@@
 F 2 "Resistor_SMD:R_0805_2012Metric" V 5180 6750 50  0001 C CNN
 F 3 "~" H 5250 6750 50  0001 C CNN
+F 4 "C17414" H 5250 6750 50  0001 C CNN "LCSC"
 	1    5250 6750
 	1    0    0    -1
@@
 F 2 "Resistor_SMD:R_0805_2012Metric" V 5080 6750 50  0001 C CNN
 F 3 "~" H 5150 6750 50  0001 C CNN
+F 4 "C17414" H 5150 6750 50  0001 C CNN "LCSC"
 	1    5150 6750
 	-1   0    0    1
@@
 F 2 "fuse:THRMC7451X160N" H 5750 3700 50  0001 L CNN
 F 3 "~" H 5700 3900 50  0001 C CNN
+F 4 "C207091" V 5700 3900 50  0001 C CNN "LCSC"
 	1    5700 3900
 	0    1    1    0
@@
 F 2 "Package_SO:SOIC-8_3.9x4.9mm_P1.27mm" H 5850 3950 50  0001 C CNN
 F 3 "http://www.ti.com/lit/ds/symlink/ina219.pdf" H 5400 4200 50  0001 C CNN
+F 4 "C138706" V 5050 4300 50  0001 C CNN "LCSC"
 	1    5050 4300
 	0    1    1    0
@@
 AR Path="/5E5E123A" Ref="R2"  Part="1"
 F 0 "R2" V 4843 3800 50  0000 C CNN
-F 1 "0.02" V 4934 3800 50  0000 C CNN
-F 2 "Resistor_SMD:R_2010_5025Metric" V 4980 3800 50  0001 C CNN
+F 1 "0.02 1W" V 4934 3800 50  0000 C CNN
+F 2 "Resistor_SMD:R_2512_6332Metric" V 4980 3800 50  0001 C CNN
 F 3 "~" H 5050 3800 50  0001 C CNN
+F 4 "C127705" V 5050 3800 50  0001 C CNN "LCSC"
 	1    5050 3800
 	0    1    1    0
@@
 F 2 "Resistor_SMD:R_0805_2012Metric" V 5180 4950 50  0001 C CNN
 F 3 "~" H 5250 4950 50  0001 C CNN
+F 4 "C17414" H 5250 4950 50  0001 C CNN "LCSC"
 	1    5250 4950
 	1    0    0    -1
@@
 F 2 "Resistor_SMD:R_0805_2012Metric" V 5080 4950 50  0001 C CNN
 F 3 "~" H 5150 4950 50  0001 C CNN
+F 4 "C17414" H 5150 4950 50  0001 C CNN "LCSC"
 	1    5150 4950
 	-1   0    0    1
@@
 Wire Wire Line
 	8600 5400 8850 5400
+$Comp
+L Analog_ADC:INA219AxD U?
+U 1 1 5E5E1165
+P 2250 4250
+AR Path="/5E5C0CC9/5E5E1165" Ref="U?"  Part="1"
+AR Path="/5E5E1165" Ref="U1"  Part="1"
+F 0 "U1" V 2400 4650 50  0000 C CNN
+F 1 "INA219AxD" V 2500 4750 50  0000 C CNN
+F 2 "Package_SO:SOIC-8_3.9x4.9mm_P1.27mm" H 3050 3900 50  0001 C CNN
+F 3 "http://www.ti.com/lit/ds/symlink/ina219.pdf" H 2600 4150 50  0001 C CNN
+F 4 "C138706" V 2250 4250 50  0001 C CNN "LCSC"
+	1    2250 4250
+	0    1    1    0
+$EndComp
+$Comp
+L Connector:Jack-DC J?
+U 1 1 5F50DE31
+P 9850 2250
+AR Path="/5E5C0CC9/5F50DE31" Ref="J?"  Part="1"
+AR Path="/5F50DE31" Ref="J2"  Part="1"
+F 0 "J2" H 9907 2575 50  0000 C CNN
+F 1 "Jack-DC" H 9907 2484 50  0000 C CNN
+F 2 "Connector_BarrelJack:BarrelJack_Horizontal" H 9900 2210 50  0001 C CNN
+F 3 "~" H 9900 2210 50  0001 C CNN
+	1    9850 2250
+	-1   0    0    -1
+$EndComp
+Wire Wire Line
+	8650 5550 8650 5700
+Wire Wire Line
+	8650 5550 8850 5550
 $EndSCHEMATC

Commit message: add hexa i2c adress
Other:
- note added: "I2C adres (bin): 1000001\nI2C adres (hex): 0x41"
- note added: "I2C adres (bin): 1000011\nI2C adres (hexa): 0x4d"
- note added: "I2C adres (bin): 1000100\nI2C adres (hex): 0x44"
- note added: "I2C adres (bin): 1001001\nI2C adres (hex): 0x49"
- note removed: "I2C adres : 1000001"
- note removed: "I2C adres : 1000010"
- note removed: "I2C adres : 1000011"
- note removed: "I2C adres : 1000100"
Changed lines of the file:
@@
 $EndComp
 Text Notes 2800 6600 0    50   ~ 0
-I2C adres : 1000011
+I2C adres (bin): 1000011\nI2C adres (hexa): 0x4d
 $Comp
 L Connector_Generic:Conn_01x02 J?
@@
 $EndComp
 Text Notes 2750 4750 0    50   ~ 0
-I2C adres : 1000001
+I2C adres (bin): 1000001\nI2C adres (hex): 0x41
 $Comp
 L Connector_Generic:Conn_01x02 J?
@@
 $EndComp
 Text Notes 5550 6600 0    50   ~ 0
-I2C adres : 1000100
+I2C adres (bin): 1000100\nI2C adres (hex): 0x44
 $Comp
 L Connector_Generic:Conn_01x02 J?
@@
 $EndComp
 Text Notes 5550 4800 0    50   ~ 0
-I2C adres : 1000010
+I2C adres (bin): 1001001\nI2C adres (hex): 0x49
 Wire Wire Line
 	5250 4750 4950 4750

Commit message: change DC for XT30, change controle res for pwm
add ds1050Z-025+ change for xt30 connector for in alim
Parts:
- removed D1: B140HW-7, Diode_SMD:D_SOD-123, symbol Device:D
- removed F1: Polyfuse_Small, fuse:FUSC3216X100N, symbol Device:Polyfuse_Small
- added Q1: IRFS7530TRLPBF, Package_TO_SOT_SMD:TO-263-2, symbol Transistor_FET:IRF540N
- added R13: 1k, Resistor_SMD:R_0805_2012Metric, symbol Device:R
- J2: footprint Connector_BarrelJack:BarrelJack_Horizontal -> Connector_AMASS:AMASS_XT30PW-M_1x02_P2.50mm_Horizontal
- MK1, MK2, MK3, MK4: footprint MountingHole:MountingHole_2.7mm_M2.5 -> MountingHole:MountingHole_3.2mm_M3
Connections:
- net +12V: now also R13.1
- net GND: now also Q1.3 (S); no longer J1.2 (Pin_2), J1.3 (Pin_3), J2.2
- new net: Q1.1 (G), R13.2
- new net gnd_no: J1.2 (Pin_2), J1.3 (Pin_3), J2.2, Q1.2 (D)
Other:
- note added: "Polarity protection"
Changed lines of the file:
@@
 F 0 "MK1" H 4850 1096 50  0000 L CNN
 F 1 "M2.5" H 4850 1005 50  0000 L CNN
-F 2 "MountingHole:MountingHole_2.7mm_M2.5" H 4750 1050 60  0001 C CNN
+F 2 "MountingHole:MountingHole_3.2mm_M3" H 4750 1050 60  0001 C CNN
 F 3 "" H 4750 1050 60  0001 C CNN
 	1    4750 1050
@@
 F 0 "MK3" H 5300 1096 50  0000 L CNN
 F 1 "M2.5" H 5300 1005 50  0000 L CNN
-F 2 "MountingHole:MountingHole_2.7mm_M2.5" H 5200 1050 60  0001 C CNN
+F 2 "MountingHole:MountingHole_3.2mm_M3" H 5200 1050 60  0001 C CNN
 F 3 "" H 5200 1050 60  0001 C CNN
 	1    5200 1050
@@
 F 0 "MK2" H 4850 1296 50  0000 L CNN
 F 1 "M2.5" H 4850 1205 50  0000 L CNN
-F 2 "MountingHole:MountingHole_2.7mm_M2.5" H 4750 1250 60  0001 C CNN
+F 2 "MountingHole:MountingHole_3.2mm_M3" H 4750 1250 60  0001 C CNN
 F 3 "" H 4750 1250 60  0001 C CNN
 	1    4750 1250
@@
 F 0 "MK4" H 5300 1296 50  0000 L CNN
 F 1 "M2.5" H 5300 1205 50  0000 L CNN
-F 2 "MountingHole:MountingHole_2.7mm_M2.5" H 5200 1250 60  0001 C CNN
+F 2 "MountingHole:MountingHole_3.2mm_M3" H 5200 1250 60  0001 C CNN
 F 3 "" H 5200 1250 60  0001 C CNN
 	1    5200 1250
@@
 	0    1    1    0
 $EndComp
-$Comp
-L Connector:Screw_Terminal_01x04 J1
-U 1 1 5E5C712D
-P 9650 4200
-F 0 "J1" H 9730 4192 50  0000 L CNN
-F 1 "Screw_Terminal_01x04" H 9730 4101 50  0000 L CNN
-F 2 "TerminalBlock:TerminalBlock_bornier-4_P5.08mm" H 9650 4200 50  0001 C CNN
-F 3 "~" H 9650 4200 50  0001 C CNN
-	1    9650 4200
-	1    0    0    -1
-$EndComp
-$Comp
-L power:GND #PWR0101
-U 1 1 5E5C7133
-P 8850 2350
-F 0 "#PWR0101" H 8850 2100 50  0001 C CNN
-F 1 "GND" V 8855 2222 50  0000 R CNN
-F 2 "" H 8850 2350 50  0001 C CNN
-F 3 "" H 8850 2350 50  0001 C CNN
-	1    8850 2350
-	0    1    -1   0
-$EndComp
-$Comp
-L power:GND #PWR0103
-U 1 1 5E5C713F
-P 9400 4250
-F 0 "#PWR0103" H 9400 4000 50  0001 C CNN
-F 1 "GND" V 9405 4122 50  0000 R CNN
-F 2 "" H 9400 4250 50  0001 C CNN
-F 3 "" H 9400 4250 50  0001 C CNN
-	1    9400 4250
-	0    1    1    0
-$EndComp
 Wire Wire Line
 	9450 4200 9400 4200
 Wire Wire Line
-	9400 4200 9400 4250
-Wire Wire Line
-	9400 4250 9400 4300
-Wire Wire Line
 	9400 4300 9450 4300
-Connection ~ 9400 4250
 $Comp
 L power:VCC #PWR0104
@@
 	1    0    0    -1
 $EndComp
-$Comp
-L power:+12V #PWR0105
-U 1 1 5E5C7150
-P 9450 4400
-F 0 "#PWR0105" H 9450 4250 50  0001 C CNN
-F 1 "+12V" H 9465 4573 50  0000 C CNN
-F 2 "" H 9450 4400 50  0001 C CNN
-F 3 "" H 9450 4400 50  0001 C CNN
-	1    9450 4400
-	-1   0    0    1
-$EndComp
-Wire Wire Line
-	9550 2350 9150 2350
-$Comp
-L Device:D D1
-U 1 1 5E5C7165
-P 9150 2200
-F 0 "D1" V 9104 2279 50  0000 L CNN
-F 1 "B140HW-7" V 9195 2279 50  0000 L CNN
-F 2 "Diode_SMD:D_SOD-123" H 9150 2200 50  0001 C CNN
-F 3 "~" H 9150 2200 50  0001 C CNN
-F 4 "C134429" V 9150 2200 50  0001 C CNN "LCSC"
-	1    9150 2200
-	0    1    1    0
-$EndComp
-Connection ~ 9150 2350
-Wire Wire Line
-	9150 2350 8850 2350
-$Comp
-L Device:Polyfuse_Small F1
-U 1 1 5E5C716D
-P 9150 1950
-F 0 "F1" H 9250 1900 50  0000 L CNN
-F 1 "Polyfuse_Small" H 8550 1900 50  0000 L CNN
-F 2 "fuse:FUSC3216X100N" H 9200 1750 50  0001 L CNN
-F 3 "~" H 9150 1950 50  0001 C CNN
-F 4 "C151162" H 9150 1950 50  0001 C CNN "LCSC"
-	1    9150 1950
-	1    0    0    -1
-$EndComp
 Wire Wire Line
 	9550 2150 9550 1850
-Wire Wire Line
-	9550 1850 9150 1850
-Wire Wire Line
-	9150 1850 8850 1850
-Connection ~ 9150 1850
-$Comp
-L power:+12V #PWR0110
-U 1 1 5E5C7177
-P 8850 1850
-F 0 "#PWR0110" H 8850 1700 50  0001 C CNN
-F 1 "+12V" V 8865 1978 50  0000 L CNN
-F 2 "" H 8850 1850 50  0001 C CNN
-F 3 "" H 8850 1850 50  0001 C CNN
-	1    8850 1850
-	0    -1   -1   0
-$EndComp
 $Comp
 L Device:CP C1
@@
 	0    1    1    0
 $EndComp
+Wire Wire Line
+	8650 5550 8650 5700
+Wire Wire Line
+	8650 5550 8850 5550
+$Comp
+L Transistor_FET:IRF540N Q1
+U 1 1 5F94BD9C
+P 7350 2650
+F 0 "Q1" V 7599 2650 50  0000 C CNN
+F 1 "IRFS7530TRLPBF" V 7690 2650 50  0000 C CNN
+F 2 "Package_TO_SOT_SMD:TO-263-2" H 7600 2575 50  0001 L CIN
+F 3 "http://www.irf.com/product-info/datasheets/data/irf540n.pdf" H 7350 2650 50  0001 L CNN
+F 4 "C500544" V 7350 2650 50  0001 C CNN "LCSC"
+	1    7350 2650
+	0    1    1    0
+$EndComp
+$Comp
+L Connector:Screw_Terminal_01x04 J1
+U 1 1 5E5C712D
+P 9650 4200
+F 0 "J1" H 9730 4192 50  0000 L CNN
+F 1 "Screw_Terminal_01x04" H 9730 4101 50  0000 L CNN
+F 2 "TerminalBlock:TerminalBlock_bornier-4_P5.08mm" H 9650 4200 50  0001 C CNN
+F 3 "~" H 9650 4200 50  0001 C CNN
+	1    9650 4200
+	1    0    0    -1
+$EndComp
+Wire Wire Line
+	8850 2350 9550 2350
+Wire Wire Line
+	8850 1850 9550 1850
+$Comp
+L power:+12V #PWR0101
+U 1 1 5F9723E9
+P 7350 2150
+F 0 "#PWR0101" H 7350 2000 50  0001 C CNN
+F 1 "+12V" V 7365 2278 50  0000 L CNN
+F 2 "" H 7350 2150 50  0001 C CNN
+F 3 "" H 7350 2150 50  0001 C CNN
+	1    7350 2150
+	1    0    0    -1
+$EndComp
+$Comp
+L Device:R R13
+U 1 1 5F972BB9
+P 7350 2300
+F 0 "R13" H 7420 2346 50  0000 L CNN
+F 1 "1k" V 7350 2250 50  0000 L CNN
+F 2 "Resistor_SMD:R_0805_2012Metric" V 7280 2300 50  0001 C CNN
+F 3 "~" H 7350 2300 50  0001 C CNN
+	1    7350 2300
+	1    0    0    -1
+$EndComp
+Text Label 8850 2350 2    50   ~ 0
+gnd_no
+$Comp
+L power:+12V #PWR0102
+U 1 1 5F98CD3F
+P 8850 1850
+F 0 "#PWR0102" H 8850 1700 50  0001 C CNN
+F 1 "+12V" V 8865 1978 50  0000 L CNN
+F 2 "" H 8850 1850 50  0001 C CNN
+F 3 "" H 8850 1850 50  0001 C CNN
+	1    8850 1850
+	0    -1   -1   0
+$EndComp
+Wire Wire Line
+	9400 4200 9400 4300
+$Comp
+L power:+12V #PWR0103
+U 1 1 5F9A75CB
+P 9450 4400
+F 0 "#PWR0103" H 9450 4250 50  0001 C CNN
+F 1 "+12V" H 9465 4573 50  0000 C CNN
+F 2 "" H 9450 4400 50  0001 C CNN
+F 3 "" H 9450 4400 50  0001 C CNN
+	1    9450 4400
+	-1   0    0    1
+$EndComp
+Text Label 7550 2750 0    50   ~ 0
+gnd_no
+$Comp
+L power:GND #PWR0105
+U 1 1 5F9B3CAE
+P 7150 2750
+F 0 "#PWR0105" H 7150 2500 50  0001 C CNN
+F 1 "GND" V 7155 2622 50  0000 R CNN
+F 2 "" H 7150 2750 50  0001 C CNN
+F 3 "" H 7150 2750 50  0001 C CNN
+	1    7150 2750
+	0    1    1    0
+$EndComp
+Text Label 9400 4250 2    50   ~ 0
+gnd_no
+Wire Notes Line
+	6650 1600 8100 1600
+Wire Notes Line
+	8100 1600 8100 3250
+Wire Notes Line
+	8100 3250 6650 3250
+Wire Notes Line
+	6650 3250 6650 1600
+Text Notes 6700 1700 0    50   ~ 0
+Polarity protection
 $Comp
 L Connector:Jack-DC J?
@@
 F 0 "J2" H 9907 2575 50  0000 C CNN
 F 1 "Jack-DC" H 9907 2484 50  0000 C CNN
-F 2 "Connector_BarrelJack:BarrelJack_Horizontal" H 9900 2210 50  0001 C CNN
+F 2 "Connector_AMASS:AMASS_XT30PW-M_1x02_P2.50mm_Horizontal" H 9900 2210 50  0001 C CNN
 F 3 "~" H 9900 2210 50  0001 C CNN
 	1    9850 2250
 	-1   0    0    -1
 $EndComp
-Wire Wire Line
-	8650 5550 8650 5700
-Wire Wire Line
-	8650 5550 8850 5550
 $EndSCHEMATC

Commit message: add serigraph and update name for componant
Parts:
- F2, F3, F4, F5: value Polyfuse_Small -> 2920L330/24; LCSC C207091 -> (none)
- J2: value Jack-DC -> XT30
- MK1, MK2, MK3, MK4: value M2.5 -> M3
Changed lines of the file:
@@
 P 4750 1050
 F 0 "MK1" H 4850 1096 50  0000 L CNN
-F 1 "M2.5" H 4850 1005 50  0000 L CNN
+F 1 "M3" H 4850 1005 50  0000 L CNN
 F 2 "MountingHole:MountingHole_3.2mm_M3" H 4750 1050 60  0001 C CNN
 F 3 "" H 4750 1050 60  0001 C CNN
@@
 P 5200 1050
 F 0 "MK3" H 5300 1096 50  0000 L CNN
-F 1 "M2.5" H 5300 1005 50  0000 L CNN
+F 1 "M3" H 5300 1005 50  0000 L CNN
 F 2 "MountingHole:MountingHole_3.2mm_M3" H 5200 1050 60  0001 C CNN
 F 3 "" H 5200 1050 60  0001 C CNN
@@
 P 4750 1250
 F 0 "MK2" H 4850 1296 50  0000 L CNN
-F 1 "M2.5" H 4850 1205 50  0000 L CNN
+F 1 "M3" H 4850 1205 50  0000 L CNN
 F 2 "MountingHole:MountingHole_3.2mm_M3" H 4750 1250 60  0001 C CNN
 F 3 "" H 4750 1250 60  0001 C CNN
@@
 P 5200 1250
 F 0 "MK4" H 5300 1296 50  0000 L CNN
-F 1 "M2.5" H 5300 1205 50  0000 L CNN
+F 1 "M3" H 5300 1205 50  0000 L CNN
 F 2 "MountingHole:MountingHole_3.2mm_M3" H 5200 1250 60  0001 C CNN
 F 3 "" H 5200 1250 60  0001 C CNN
@@
 AR Path="/5E5E1105" Ref="F4"  Part="1"
 F 0 "F4" V 2745 5700 50  0000 C CNN
-F 1 "Polyfuse_Small" V 2836 5700 50  0000 C CNN
+F 1 "2920L330/24" V 2836 5700 50  0000 C CNN
 F 2 "fuse:THRMC7451X160N" H 3000 5500 50  0001 L CNN
 F 3 "~" H 2950 5700 50  0001 C CNN
-F 4 "C207091" V 2950 5700 50  0001 C CNN "LCSC"
+F 4 "" V 2950 5700 50  0001 C CNN "LCSC"
 	1    2950 5700
 	0    1    1    0
@@
 AR Path="/5E5E115F" Ref="F2"  Part="1"
 F 0 "F2" V 2695 3850 50  0000 C CNN
-F 1 "Polyfuse_Small" V 2786 3850 50  0000 C CNN
+F 1 "2920L330/24" V 2786 3850 50  0000 C CNN
 F 2 "fuse:THRMC7451X160N" H 2950 3650 50  0001 L CNN
 F 3 "~" H 2900 3850 50  0001 C CNN
-F 4 "C207091" V 2900 3850 50  0001 C CNN "LCSC"
+F 4 "" V 2900 3850 50  0001 C CNN "LCSC"
 	1    2900 3850
 	0    1    1    0
@@
 AR Path="/5E5E11BF" Ref="F5"  Part="1"
 F 0 "F5" V 5495 5700 50  0000 C CNN
-F 1 "Polyfuse_Small" V 5586 5700 50  0000 C CNN
+F 1 "2920L330/24" V 5586 5700 50  0000 C CNN
 F 2 "fuse:THRMC7451X160N" H 5750 5500 50  0001 L CNN
 F 3 "~" H 5700 5700 50  0001 C CNN
-F 4 "C207091" V 5700 5700 50  0001 C CNN "LCSC"
+F 4 "" V 5700 5700 50  0001 C CNN "LCSC"
 	1    5700 5700
 	0    1    1    0
@@
 AR Path="/5E5E121F" Ref="F3"  Part="1"
 F 0 "F3" V 5495 3900 50  0000 C CNN
-F 1 "Polyfuse_Small" V 5586 3900 50  0000 C CNN
+F 1 "2920L330/24" V 5586 3900 50  0000 C CNN
 F 2 "fuse:THRMC7451X160N" H 5750 3700 50  0001 L CNN
 F 3 "~" H 5700 3900 50  0001 C CNN
-F 4 "C207091" V 5700 3900 50  0001 C CNN "LCSC"
+F 4 "" V 5700 3900 50  0001 C CNN "LCSC"
 	1    5700 3900
 	0    1    1    0
@@
 AR Path="/5F50DE31" Ref="J2"  Part="1"
 F 0 "J2" H 9907 2575 50  0000 C CNN
-F 1 "Jack-DC" H 9907 2484 50  0000 C CNN
+F 1 "XT30" H 9907 2484 50  0000 C CNN
 F 2 "Connector_AMASS:AMASS_XT30PW-M_1x02_P2.50mm_Horizontal" H 9900 2210 50  0001 C CNN
 F 3 "~" H 9900 2210 50  0001 C CNN
